File: PCB/PCB.kicad_pcb (KiCad board)
At the start: 2 copper layers, 100 x 100 mm, 103 parts, among them J1 USB_B_Mini, J2 Screw_Terminal_01x02, J3 Conn_01x03, K1 G6K-2, Q1 IPD50R3K0CE, Q2 2N7002, SW1 SW_Omron_B3FS, U1 STM32F373C8Tx, U2 LIS3MDL, U3 INA848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

Commit message: Updated
Parts:
- C19, C25: value C_Small -> 100nF
- C20, C21: value C_Small -> 10nF
- C22: value C_Small -> 220pF
- D6: value D_Schottky -> SD101A
- D7: value 1.5KExxA -> SD101A
- R10, R9: value R_Small -> 49.9h
Connections:
- U1 pad 13: unconnected-(U1-PA3-Pad13) -> EN_{B}
Routing:
- net EN_{B}: track 1.97 -> 90.8 mm, vias 0 -> 4
- net GNDD: vias 318 -> 334
